File: PCB/V3/QNOB_V5/QNOB_V5.kicad_sch (KiCad schematic)
At the start: 16 parts, among them J1 Conn_01x05, J2 Conn_01x05, U1 ESP32-C3_SUPERMINI

Commit message: move versions
Parts:
- removed JP2, JP4: SolderJumper_3_Open, Jumper:SolderJumper-3_P1.3mm_Open_RoundedPad1.0x1.5mm, symbol Jumper:SolderJumper_3_Open
Other:
- removed sheet RTC
- note removed: "Encoder mode selector"
