File: ScreenBase_V2/ScreenBase_V2.kicad_pcb (KiCad board)
At the start: 2 copper layers, 44 x 42 mm, 24 parts, among them J1 Connector_PinHeader_2.54mm:Pi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, J10 Conn_01x01_Pin, J11 Conn_01x01_Pin, J12 Conn_01x01_Pin, J13 Conn_01x01_Pin, J14 Conn_01x01_Pin, J15 Conn_01x01_Pin, J16 Conn_01x01_Pin, J17 Conn_01x01_Pin, J18 Conn_01x01_Pin, J2 Connector_PinHeader_2.54mm:Pi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, J3 Conn_01x01_Pin, J4 Conn_01x01_Pin, J5 Conn_01x01_Pin, J6 Conn_01x01_Pin, J7 Conn_01x01_Pin, J8 Conn_01x01_Pin, J9 Conn_01x01_Pin, U1 BME688

Commit message: start refactor
Parts:
- J1, J2: footprint Connector_PinHeader_2.54mm:PinHeader_2x04_P2.54mm_Vertical_SMD -> Connector_PinHeader_2.54mm:PinHeader_2x04_P2.54mm_Vertical
- moved J1 119.9 mm to (-17.8, -3.31)
- moved J2 119.9 mm to (15.2, -3.31)
- moved C2 117.1 mm to (16.8, -7.50)
- moved J11 116.7 mm to (-9.20, 1.60)
- moved J12 116.7 mm to (-9.20, 3.40)
- moved J13 116.7 mm to (-9.20, -7.40)
- moved J14 116.7 mm to (-9.20, -3.80)
- moved J15 116.7 mm to (-9.20, -0.20)
- moved J16 116.7 mm to (-9.20, 5.00)
- moved J6 116.7 mm to (-9.20, -2.00)
- moved J9 116.7 mm to (-9.20, -5.60)
- moved C1 116.7 mm to (-16.5, -8.00)
- moved C3 116.7 mm to (-8.25, -17.5)
- moved C4 116.7 mm to (-8.25, -15.5)
- moved J10 116.7 mm to (9.20, -4.40)
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Routing:
- net Net-(J17-Pin_1): track 10.7 -> 7.66 mm
- net /SCL: track 23.2 -> 26.1 mm
- net /GPIO2: track 8.48 -> 10.6 mm
- net +BATT: track 5.04 -> 6.39 mm
- net /GPIO9: track 10.5 -> 11.8 mm, vias 0 -> 1
- net /SDA: track 23.2 -> 24.4 mm, vias 0 -> 2
- net 5V: track 6.50 -> 5.37 mm
- net 3V3: track 33.2 -> 34.3 mm
- net /GPIO16: track 8.45 -> 9.48 mm
- net /GPIO1: track 5.91 -> 6.42 mm
- net GND: vias 47 -> 46
Other:
- board text added: "0"
- board text added: "1"
- board text added: "15"
- board text added: "16"
- board text added: "17"
- board text added: "2"
- board text added: "3v3"
- board text added: "5V"
- board text added: "9"
- board text added: "BATT+"
- board text added: "GND"
- board text added: "SCL"
- board text added: "SDA"
- board text removed: "Blue"
- board text removed: "Green"
- board text removed: "Grey"
- board text removed: "Orange"
- board text removed: "Pink"
- board text removed: "Purple"
- board text removed: "White"
- board text removed: "Yellow"
